Commit message: lecture 3 - adding laser scan

File: simulation_ws/src/robot_description/urdf/gazebo.xacro (robot description, xacro)
@@ -27,3 +27,37 @@
     </plugin>
   </gazebo>
+  <!-- Adding sensor behavior to laser link -->
+  <gazebo reference="sensor_laser">
+    <sensor type="ray" name="head_hokuyo_sensor">
+    <!-- <sensor type="gpu_ray" name="head_hokuyo_sensor"> -->
+      <pose>0 0 0 0 0 0</pose>
+      <visualize>false</visualize>
+      <update_rate>20</update_rate>
+      <ray>
+        <scan>
+          <horizontal>
+            <samples>720</samples>
+            <resolution>1</resolution>
+            <min_angle>-1.570796</min_angle>
+            <max_angle>1.570796</max_angle>
+          </horizontal>
+        </scan>
+        <range>
+          <min>0.10</min>
+          <max>10.0</max>
+          <resolution>0.01</resolution>
+        </range>
+        <noise>
+          <type>gaussian</type>
+          <mean>0.0</mean>
+          <stddev>0.01</stddev>
+        </noise>
+      </ray>
+      <plugin name="gazebo_ros_head_hokuyo_controller" filename="libgazebo_ros_laser.so">
+      <!-- <plugin name="gazebo_ros_head_hokuyo_controller" filename="libgazebo_ros_gpu_laser.so"> -->
+        <topicName>/robot/laser/scan</topicName>
+        <frameName>sensor_laser</frameName>
+      </plugin>
+    </sensor>
+  </gazebo>
 </robot>

File: simulation_ws/src/robot_description/urdf/macro.xacro (robot description, xacro)
@@ -32,3 +32,7 @@
     </joint>
   </xacro:macro>
+  <xacro:macro name="cylinder_inertia" params="mass r l">
+    <inertia ixx="${mass*(3*r*r+l*l)/12}" ixy = "0" ixz = "0"
+              iyy="${mass*(3*r*r+l*l)/12}" iyz = "0" izz="${mass*(r*r)/2}" />
+  </xacro:macro>
 </robot>

File: simulation_ws/src/robot_description/urdf/robot.xacro (robot description, xacro)
@@ -50,4 +50,31 @@
     </visual>
   </link>
+  <!-- Link for laser -->
+  <link name="sensor_laser">
+    <inertial>
+      <origin xyz="0 0 0" rpy="0 0 0" />
+      <mass value="1" />
+      <xacro:cylinder_inertia mass="1" r="0.05" l="0.1" />
+    </inertial>
+    <visual>
+      <origin xyz="0 0 0" rpy="0 0 0" />
+      <geometry>
+        <cylinder radius="0.05" length="0.1"/>
+      </geometry>
+      <material name="white" />
+    </visual>
+    <collision>
+      <origin xyz="0 0 0" rpy="0 0 0"/>
+      <geometry>
+        <cylinder radius="0.05" length="0.1"/>
+      </geometry>
+    </collision>
+  </link>
+  <!-- Joint for laser -->
+  <joint name="joint_sensor_laser" type="fixed">
+    <origin xyz="0.15 0 0.05" rpy="0 0 0"/>
+    <parent link="link_chassis"/>
+    <child link="sensor_laser"/>
+  </joint>
   <!-- Right Wheel Link -->
   <xacro:link_wheel name="link_right_wheel" />

Commit message: lecture 5 - obstacle avoidance

File: simulation_ws/src/robot_description/urdf/gazebo.xacro (robot description, xacro)
@@ -32,18 +32,19 @@
     <!-- <sensor type="gpu_ray" name="head_hokuyo_sensor"> -->
       <pose>0 0 0 0 0 0</pose>
-      <visualize>false</visualize>
-      <update_rate>20</update_rate>
+      <visualize>1</visualize>
+      <always_on>1</always_on>
+      <update_rate>30</update_rate>
       <ray>
         <scan>
           <horizontal>
-            <samples>720</samples>
+            <samples>10</samples>
             <resolution>1</resolution>
-            <min_angle>-1.570796</min_angle>
-            <max_angle>1.570796</max_angle>
+            <min_angle>-1.0472</min_angle>
+            <max_angle>1.0472</max_angle>
           </horizontal>
         </scan>
         <range>
           <min>0.10</min>
-          <max>10.0</max>
+          <max>3.0</max>
           <resolution>0.01</resolution>
         </range>

File: simulation_ws/src/robot_description/urdf/materials.xacro (robot description, xacro)
@@ -25,3 +25,14 @@
     <color rgba="1.0 1.0 1.0 1.0"/>
   </material>
+  <material name="laserLight">
+    <lighting>1</lighting>
+    <ambient>0.3 0.3 0.3 1</ambient>
+    <diffuse>0.7 0.7 0.7 1</diffuse>
+    <specular>0.01 0.01 0.01 1</specular>
+    <emissive>0 0 0 1</emissive>
+  </material>
+  <material name="collisionLaser">
+    <laser_retro>0</laser_retro>
+    <max_contacts>10</max_contacts>
+  </material>
 </robot>

File: simulation_ws/src/robot_description/urdf/robot.xacro (robot description, xacro)
@@ -54,5 +54,5 @@
     <inertial>
       <origin xyz="0 0 0" rpy="0 0 0" />
-      <mass value="1" />
+      <mass value="4" />
       <xacro:cylinder_inertia mass="1" r="0.05" l="0.1" />
     </inertial>
@@ -63,4 +63,5 @@
       </geometry>
       <material name="white" />
+      <material name="laserLight" />
     </visual>
     <collision>
@@ -69,4 +70,5 @@
         <cylinder radius="0.05" length="0.1"/>
       </geometry>
+      <material name="collisionLaser" />
     </collision>
   </link>
